Commit message: New codes commit message

File: urdf/cartpole.urdf (robot description, URDF)
Before this commit: robot physics, 3 links, 2 joints
Links:
- link pole: mass 0.1 -> 10

Commit message: almpst finalised c0de

File: urdf/cartpole.urdf (robot description, URDF)
Before this commit: robot physics, 3 links, 2 joints
Links:
- link pole: mass 10 -> 0.1; geometry collision cylinder length=1.0 radius=0.03; visual box size=0.05 0.05 1.0
Joints:
- joint slider_to_cart: limit lower=-15 upper=15 effort=1000.0 velocity=5 -> lower=-2.4 upper=2.4 effort=50.0 velocity=1.5

File: urdf/invertedpendulum.urdf (robot description, URDF)
Before this commit: robot cart_pole_with_wheels, 4 links, 3 joints
Links:
- link left_wheel: geometry collision cylinder length=0.05 radius=0.1; visual cylinder length=0.05 radius=0.1
- link right_wheel: geometry collision cylinder length=0.05 radius=0.1; visual cylinder length=0.05 radius=0.1

Commit message: new commits

File: urdf/cartpole.urdf (robot description, URDF)
Before this commit: robot physics, 3 links, 2 joints
Links:
- link cart: mass 1 -> 4
- link pole: mass 0.1 -> 1

File: urdf/walker.urdf (robot description, URDF)
Before this commit: robot assistive_walker, 5 links, 4 joints
Links:
- link base_link: geometry collision box size=0.3 0.5 0.24; visual box size=0.3 0.5 0.24
Joints:
- joint imu_joint: origin xyz=0 0 0.2 rpy=0 0 0 -> xyz=0 0 0.24 rpy=0 0 0
- joint left_wheel_joint: origin xyz=0 0.18 0.08 rpy=0 0 0 -> xyz=0 0.28 0 rpy=0 0 0
- joint pole_joint: origin xyz=0.18 0 0.24 rpy=0 0 0 -> xyz=0.05 0 0.24 rpy=0 0 0; type fixed -> revolute
- joint right_wheel_joint: origin xyz=0 -0.18 0.08 rpy=0 0 0 -> xyz=0 -0.28 0 rpy=0 0 0
