Commit message: Some new code

File: urdf/walker.urdf (robot description, URDF)
Before this commit: robot assistive_walker, 5 links, 4 joints
Joints:
- joint pole_joint: limit (none) -> lower=-3.14 upper=3.14 effort=10 velocity=10

Commit message: main main

File: urdf/walker.urdf (robot description, URDF)
Before this commit: robot assistive_walker, 5 links, 4 joints
Joints:
- joint pole_joint: axis (none) -> 0 1 0

Commit message: some final changes

File: urdf/walker.urdf (robot description, URDF)
Before this commit: robot assistive_walker, 5 links, 4 joints
Links:
- link base_link: geometry collision box size=0.3 0.50 0.24; visual box size=0.3 0.50 0.24

Commit message: commit

File: urdf/walker.urdf (robot description, URDF)
Before this commit: robot assistive_walker, 5 links, 4 joints
Joints:
- joint left_wheel_joint: limit (none) -> effort=5.0 velocity=10.0
- joint right_wheel_joint: limit (none) -> effort=5.0 velocity=10.0
